Commit message: second update

File: pinnabot_description/urdf/Pinna_bot.xacro (robot description, xacro)
@@ -6,11 +6,15 @@
   <xacro:include filename="$(find pinnabot_description)/urdf/macros.xacro" />
   <!--Links o partes Chasis-->
+    <link name="link_chassis_root">
+    <pose>0 0 0.1 0 0 0</pose>
+    </link>
     <link name="link_chassis">
-        <!-- pose and inertial -->
+        <!-- pose -->
         <pose>0 0 0.1 0 0 0</pose>
-        <inertial>
-            <mass value="3.0"/>
+        <!--inertial -->
+        <inertial>
+            <mass value="1.8"/>
             <origin rpy="0 0 0" xyz="0 0 0"/>
-            <inertia ixx="0.0655" ixy="0" ixz="0" iyy="0.0517" iyz="0" izz="0.14"/>
+            <inertia ixx="0.0655" ixy="0.0" ixz="0.0" iyy="0.0517" iyz="0.0" izz="0.14"/>
         </inertial>
         <!--Chasis -->
@@ -31,5 +35,5 @@
     <link name="link_caster_wheel">
         <inertial>
-            <mass value="0.15"/>
+            <mass value="0.1"/>
             <inertia ixx="0.001107" ixy="0" ixz="0" iyy="0.001107" iyz="0" izz="0.002152"/>
         </inertial>
@@ -49,5 +53,5 @@
     <link name="link_caster_axis_support">
         <inertial>
-            <mass value="0.08"/>
+            <mass value="0.03"/>
             <inertia ixx="1e-6" ixy="0" ixz="0" iyy="1e-6" iyz="0" izz="1e-6" />
         </inertial>
@@ -86,5 +90,5 @@
     <link name="link_wheel_right">
         <inertial>
-            <mass value="1.0"/>
+            <mass value="0.80"/>
             <origin rpy="0 1.5707 0" xyz="0 0 0"/>
             <inertia ixx="0.01107" ixy="0" ixz="0" iyy="0.01107" iyz="0" izz="0.02152"/>
@@ -105,5 +109,5 @@
     <link name="link_wheel_left">
         <inertial>
-            <mass value="1.0"/>
+            <mass value="0.80"/>
             <origin rpy="0 -1.5707 0" xyz="0 0 0"/>
             <inertia ixx="0.01107" ixy="0" ixz="0" iyy="0.01107" iyz="0" izz="0.02152"/>
@@ -148,5 +152,5 @@
     <link name="module_jetson_link">
       <inertial>
-        <mass value="0.4"/>
+        <mass value="0.1"/>
         <inertia ixx="0.0" ixy="0.0" ixz="0.0" iyy="0.0" iyz="0.0" izz="0.0"/>
       </inertial>
@@ -181,5 +185,5 @@
     <link name="sonar_front_link">
       <inertial>
-        <mass value="0.001" />
+        <mass value="0.01" />
         <origin xyz="0 0 0" rpy="0 0 0" />
         <inertia ixx="0.000000017" ixy="0" ixz="0" iyy="0.000000017" iyz="0" izz="0.000000017" />
@@ -194,5 +198,5 @@
     <link name="sonar_left_link">
       <inertial>
-        <mass value="0.001" />
+        <mass value="0.01" />
         <origin xyz="0 0 0" rpy="0 0 0" />
         <inertia ixx="0.000000017" ixy="0" ixz="0" iyy="0.000000017" iyz="0" izz="0.000000017" />
@@ -207,5 +211,5 @@
     <link name="sonar_right_link">
       <inertial>
-        <mass value="0.001" />
+        <mass value="0.01" />
         <origin xyz="0 0 0" rpy="0 0 0" />
         <inertia ixx="0.000000017" ixy="0" ixz="0" iyy="0.000000017" iyz="0" izz="0.000000017" />
@@ -219,7 +223,12 @@
     </link>
  <!--Joints o uniones-->
+    <joint name="joint_root" type="fixed">
+          <origin xyz="0 0 0" rpy="0 0 0"/>
+          <parent link="link_chassis_root" />
+          <child link="link_chassis" />
+    </joint>
     <joint name="joint_caster" type="fixed">
           <origin xyz="0 -0.1105 0.03" rpy="0 0 0"/>
-          <parent link="link_chassis" />
+          <parent link="link_chassis_root" />
           <child link="link_caster_base" />
     </joint>
@@ -243,50 +252,56 @@
           <origin rpy="0 0 0" xyz="0.122 0.085 0.023"/>
           <child link="link_wheel_right"/>
-          <parent link="link_chassis"/>
+          <parent link="link_chassis_root"/>
           <axis rpy="0 0 0" xyz="-1 0 0"/>
-          <limit effort="10000" velocity="1000"/>
           <joint_properties damping="0.80" friction="1.0"/>
+          <!-- Joint limits -->
+          <limit effort="1.76" velocity="26.2" />
+          <!-- Soft limits -->
+          <safety_controller k_velocity="10" />
     </joint>
     <joint name="joint_wheel_left" type="continuous">
           <origin rpy="0 0 0" xyz="-0.122 0.085 0.023"/>
           <child link="link_wheel_left"/>
-          <parent link="link_chassis"/>
+          <parent link="link_chassis_root"/>
           <axis rpy="0 0 0" xyz="-1 0 0"/>
-          <limit effort="10000" velocity="1000"/>
           <joint_properties damping="0.80" friction="1.0"/>
+          <!-- Joint limits -->
+          <limit effort="1.76" velocity="26.2" /> <!--effort in [N-m for revolute] & velocity in [rad/seg for revolute] is te velocity limit-->
+          <!-- Soft limits -->
+          <safety_controller k_velocity="10" />
     </joint>
     <joint name="joint_imu" type="fixed">
           <origin rpy="0 0 0" xyz="0 0.085 0.02"/>
           <child link="imu_link"/>
-          <parent link="link_chassis"/>
+          <parent link="link_chassis_root"/>
     </joint>
     <joint name="joint_camera" type="fixed">
           <origin rpy="0 0 1.57" xyz="0 0.155 0.130"/>
-          <parent link="link_chassis"/>
+          <parent link="link_chassis_root"/>
           <child link="camera_link"/>
     </joint>
     <joint name="joint_module_jetson" type="fixed">
       <origin xyz="0.0 0.0735 0.13" rpy="0.0 0.0 0.0"/>
-      <parent link="link_chassis"/>
+      <parent link="link_chassis_root"/>
       <child link="module_jetson_link"/>
     </joint>
     <joint name="joint_lidar" type="fixed">
           <origin rpy="0 0 1.5707" xyz="0 0.075 0.190"/>
-          <parent link="link_chassis"/>
+          <parent link="link_chassis_root"/>
           <child link="lidar_link"/>
     </joint>
     <joint name="joint_sonar_front" type="fixed">
       <origin xyz="0 0.158 0.051" rpy="0 0 1.5707"/>
-      <parent link="link_chassis"/>
+      <parent link="link_chassis_root"/>
       <child link="sonar_front_link"/>
     </joint>
     <joint name="joint_sonar_left" type="fixed">
       <origin xyz="-0.08 0.1405 0.051" rpy="0 0 2.1"/>
-      <parent link="link_chassis"/>
+      <parent link="link_chassis_root"/>
       <child link="sonar_left_link"/>
     </joint>
     <joint name="joint_sonar_right" type="fixed">
       <origin xyz="0.08 0.1405 0.051" rpy="0 0 1.04"/>
-      <parent link="link_chassis"/>
+      <parent link="link_chassis_root"/>
       <child link="sonar_right_link"/>
     </joint>

Commit message: change general values

File: pinnabot_description/urdf/Pinna_bot.xacro (robot description, xacro)
@@ -14,5 +14,5 @@
         <!--inertial -->
         <inertial>
-            <mass value="1.8"/>
+            <mass value="2.0"/>
             <origin rpy="0 0 0" xyz="0 0 0"/>
             <inertia ixx="0.0655" ixy="0.0" ixz="0.0" iyy="0.0517" iyz="0.0" izz="0.14"/>
@@ -35,9 +35,10 @@
     <link name="link_caster_wheel">
         <inertial>
+            <origin rpy="0 -1.57 0" xyz="0 0.0 0.0"/>
             <mass value="0.1"/>
-            <inertia ixx="0.001107" ixy="0" ixz="0" iyy="0.001107" iyz="0" izz="0.002152"/>
+            <inertia ixx="0.000009106" ixy="0" ixz="0" iyy="0.000009106" iyz="0" izz="0.000014"/>
         </inertial>
         <collision>
-          <origin rpy="0 1.57 0" xyz="0 0.00 0.0"/>
+          <origin rpy="0 1.57 0" xyz="0 0.0 0.0"/>
           <geometry>
             <cylinder length="0.019" radius="0.020"/>
@@ -90,7 +91,7 @@
     <link name="link_wheel_right">
         <inertial>
-            <mass value="0.80"/>
+            <mass value="0.08"/>
             <origin rpy="0 1.5707 0" xyz="0 0 0"/>
-            <inertia ixx="0.01107" ixy="0" ixz="0" iyy="0.01107" iyz="0" izz="0.02152"/>
+            <inertia ixx="0.00004021" ixy="0" ixz="0" iyy="0.00004021" iyz="0" izz="0.00007396"/>
         </inertial>
         <collision name="link_wheel_right_collision">
@@ -109,7 +110,7 @@
     <link name="link_wheel_left">
         <inertial>
-            <mass value="0.80"/>
+            <mass value="0.08"/>
             <origin rpy="0 -1.5707 0" xyz="0 0 0"/>
-            <inertia ixx="0.01107" ixy="0" ixz="0" iyy="0.01107" iyz="0" izz="0.02152"/>
+            <inertia ixx="0.00004021" ixy="0" ixz="0" iyy="0.00004021" iyz="0" izz="0.00007396"/>
         </inertial>
         <collision name="link_wheel_left_collision">

Commit message: Inertia chassis changes

File: pinnabot_description/urdf/Pinna_bot.xacro (robot description, xacro)
@@ -16,5 +16,5 @@
             <mass value="2.0"/>
             <origin rpy="0 0 0" xyz="0 0 0"/>
-            <inertia ixx="0.0655" ixy="0.0" ixz="0.0" iyy="0.0517" iyz="0.0" izz="0.14"/>
+            <inertia ixx="0.00049" ixy="0.0" ixz="0.0" iyy="0.00023" iyz="0.0" izz="0.0008"/>
         </inertial>
         <!--Chasis -->

Commit message: change some paremeters for experimentals tests

File: pinnabot_description/urdf/Pinna_bot.xacro (robot description, xacro)
@@ -132,4 +132,7 @@
     <!-- Camera -->
     <link name="camera_link">
+    <pose>0 0 0 1.57 0 -1.57</pose>
+    </link>
+    <link name="camera_real_link">
       <collision>
         <origin xyz="0 0 0" rpy="1.57 0 -1.57"/>
@@ -280,4 +283,9 @@
           <origin rpy="0 0 1.57" xyz="0 0.155 0.130"/>
           <parent link="link_chassis_root"/>
+          <child link="camera_real_link"/>
+    </joint>
+    <joint name="joint_camera_fake" type="fixed">
+          <origin rpy="0 -0.053 0" xyz="0 0 0"/>
+          <parent link="camera_real_link"/>
           <child link="camera_link"/>
     </joint>
